File: pcb_kicad/dap-stm32f103.kicad_pcb (KiCad board)
At the start: 2 copper layers, 35 parts, among them J1 USB_C_Receptacle_USB2.0, U1 STM32F103CBTx, Y1 SMD-5032_2P_8MHz_20ppm_20pF

Commit message: [update] pcb
Parts:
- added JTAG1: Conn_02x10_Top_Bottom, Connector_PinHeader_2.54mm:PinHeader_2x10_P2.54mm_Vertical, F.Cu at (155.4, 138.2)
- moved C3 74.9 mm to (138.7, 157.5), turned to 90 degrees
- moved D_GREEN1 71.9 mm to (128.5, 160.0), turned to 180 degrees
- moved R2 70.4 mm to (132.1, 158.0), turned to 180 degrees
- moved C2 69.7 mm to (142.2, 159.0), turned to 180 degrees
- moved D_BULE1 67.3 mm to (128.5, 158.0), turned to 180 degrees
- moved C1 64.8 mm to (145.3, 159.0)
- moved R7 63.2 mm to (138.4, 154.9)
- moved C11 63.0 mm to (138.4, 152.1), turned to 180 degrees
- moved C6 62.1 mm to (128.0, 153.7), turned to 180 degrees
- moved C7 61.7 mm to (132.1, 145.8), turned to 90 degrees
- moved R12 60.7 mm to (128.0, 148.6), turned to 180 degrees
- moved C5 59.2 mm to (130.0, 146.3), turned to 90 degrees
- moved R9 59.2 mm to (151.4, 158.5), turned to 90 degrees
- moved C13 58.8 mm to (150.9, 151.4), turned to 270 degrees
- moved R8 57.8 mm to (135.6, 157.5), turned to 90 degrees
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Routing:
- net (no net): vias 0 -> 4
Other:
- board outline added: 41.7 x 26.9 mm

Commit message: [pcb] 20%
Parts:
- removed SWD/JTAG1: Conn_02x05_Top_Bottom, Connector_PinHeader_2.54mm:PinHeader_2x05_P2.54mm_Vertical
- moved R8 11.2 mm to (146.8, 156.7), turned to 180 degrees
- moved C3 8.44 mm to (146.8, 155.2), turned to 180 degrees
- moved R9 3.06 mm to (151.1, 155.4), turned to 0 degrees
- moved C1 2.54 mm to (143.3, 160.5)
- moved C2 2.54 mm to (140.2, 160.5)
- moved Y1 2.54 mm to (141.7, 158.0)
- moved R7 2.54 mm to (141.0, 154.9)
- moved C6 1.02 mm to (128.0, 152.7)
- moved C8 1.02 mm to (128.0, 147.1)
- moved D_BULE1 0.92 mm to (127.8, 158.5)
- moved R2 0.92 mm to (131.3, 158.5)
- moved D_GREEN1 0.92 mm to (127.8, 160.5)
- moved R3 0.92 mm to (131.3, 160.5)
- moved D_RED1 0.72 mm to (141.7, 139.2)
- moved R4 0.72 mm to (145.4, 139.2)
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Routing:
- net Net-(C6-Pad1): track 0.00 -> 21.1 mm, vias 0 -> 2
- net /LED_GREEN: track 0.00 -> 20.2 mm, vias 0 -> 2
- net Net-(C8-Pad1): track 0.00 -> 19.3 mm, vias 0 -> 2
- net /LED_BULE: track 0.00 -> 18.8 mm, vias 0 -> 2
- net Net-(C5-Pad1): track 0.00 -> 10.3 mm
- net Net-(C2-Pad2): track 0.00 -> 7.63 mm
- net /TGT_USB_D+: track 0.00 -> 6.29 mm
- net Net-(C1-Pad2): track 0.00 -> 5.80 mm
- net /TGT_USB_D-: track 0.00 -> 4.73 mm
- net +3V3: track 0.00 -> 4.47 mm
- net /IF_NRESET: track 0.00 -> 3.58 mm
- net Net-(R6-Pad2): track 0.00 -> 2.47 mm
- net Net-(D_GREEN1-PadK): track 0.00 -> 2.36 mm
- net Net-(D_BULE1-PadK): track 0.00 -> 2.36 mm
Other:
- outline, holes or cut-outs redrawn

Commit message: [update] pcb 25%
Parts:
- moved R10 1.68 mm to (150.4, 155.4), turned to 0 degrees
- moved R9 1.68 mm to (150.4, 153.9), turned to 180 degrees
- moved C14 0.77 mm to (141.5, 142.1), turned to 180 degrees
- moved R5 0.25 mm to (147.1, 142.2)
Routing:
- net /IF_NRESET: track 3.58 -> 65.8 mm
- net /TGT_SWO: track 0.00 -> 18.5 mm, vias 0 -> 1
- net /TGT_NRESET: track 0.00 -> 17.5 mm
- net /TGT_SWDIO: track 0.00 -> 13.4 mm
- net /TGT_RX: track 0.00 -> 13.3 mm, vias 0 -> 1
- net /IF_SWCLK: track 0.00 -> 12.7 mm
- net /IF_SWDIO: track 0.00 -> 12.1 mm
- net /TGT_SWCLK: track 0.00 -> 7.23 mm
- net Net-(R10-Pad1): track 0.00 -> 6.08 mm
- net /LED_RED: track 0.00 -> 5.30 mm
- net Net-(D_RED1-PadA): track 0.00 -> 2.44 mm
- net Net-(C6-Pad1): track 21.1 -> 23.3 mm
- net +3V3: track 4.47 -> 6.59 mm
- net Net-(R5-Pad2): track 0.00 -> 1.95 mm

Commit message: [update] pcb 连线完成
Parts:
- moved C12 0.94 mm to (151.3, 145.0), turned to 0 degrees
- moved R1 0.70 mm to (150.9, 148.1), turned to 270 degrees
- moved C13 0.09 mm to (150.9, 151.4), turned to 90 degrees
- turned C11 to 270 degrees
Connections:
- J1 pad S1: Net-(J1-PadS1) -> GND
- JTAG1 pad 3: /TGT_NRESET -> Net-(JTAG1-Pad3)
Routing:
- net +3V3: track 6.59 -> 130.1 mm, vias 0 -> 1
- net GND: track 0.00 -> 72.2 mm, vias 0 -> 16
- net Net-(C5-Pad1): track 10.3 -> 17.9 mm
- net /TGT_SWCLK: track 7.23 -> 14.4 mm
- net Net-(R7-Pad2): track 0.00 -> 3.23 mm
Other:
- net class Default: via_dia 0.8 -> 0.6; via_drill 0.4 -> 0.3
- rule via_min_size: 0.4 -> 0.6

Commit message: [pcb] done
Parts:
- moved R4 0.36 mm to (145.7, 139.2)
Routing:
- net GND: track 72.2 -> 231.3 mm
- net Net-(C1-Pad2): track 5.80 -> 8.38 mm
- net Net-(C2-Pad2): track 7.63 -> 10.2 mm
- net /LED_RED: track 5.30 -> 6.29 mm
- added copper zone on B.Cu, net GND
- added copper zone on F.Cu, net GND
