File: pcb_kicad/dap-stm32f103.kicad_pcb (KiCad board)
At the start: 2 copper layers, 22 x 22 mm, 30 parts, among them J1 Conn_01x10, J2 Conn_01x10, J3 Conn_01x10, J4 Conn_01x10, U1 STM32F103CBTx, Y1 SMD-5032_2P_8MHz_20ppm_20pF

Commit message: [update] Gerber files
Parts:
- J1, J2, J3, J4: footprint lc_lib:stamp_2.0mm_1x10 -> lc_lib:stamp_01x10_1.27mm
- moved J3 2.14 mm to (131.8, 73.9)
- moved J4 2.02 mm to (118.0, 95.8)
- moved J2 2.00 mm to (136.0, 77.9)
- moved J1 1.91 mm to (114.0, 77.9)
Routing:
- net /STAMP_nSRESET: track 9.14 -> 6.77 mm
- net GND: track 185.3 -> 183.2 mm, vias 27 -> 29
- net /IF_NRESET: track 36.3 -> 37.3 mm
- net /PB7: track 15.6 -> 14.7 mm
- net /PB11: track 7.37 -> 8.06 mm
- net /IF_SWCLK: track 7.61 -> 8.28 mm
- net /PB6: track 13.9 -> 13.2 mm
- net /PB8: track 14.3 -> 13.7 mm
- net /PA10: track 9.36 -> 8.77 mm
- net /PC15: track 13.5 -> 12.9 mm
- net /PB5: track 13.2 -> 12.7 mm
