File: pcb_kicad/_autosave-dap-stm32f103.sch (KiCad schematic (older format))
At the start: 35 parts, among them J1 USB_C_Receptacle_USB2.0, J2 Conn_01x10, J3 Conn_01x10, J4 Conn_01x10, U1 STM32F103CBTx, Y1 SMD-5032_2P_8MHz_20ppm_20pF

Commit message: [update] stamp footprint
Parts:
- J2, J3, J4: footprint Connector_PinSocket_2.00mm:PinSocket_1x10_P2.00mm_Vertical -> lc_lib:stamp_2.0mm_1x10
Changed lines of the file:
@@
 F 0 "J2" H 9730 2792 50  0000 L CNN
 F 1 "Conn_01x10" H 9730 2701 50  0000 L CNN
-F 2 "Connector_PinSocket_2.00mm:PinSocket_1x10_P2.00mm_Vertical" H 9650 2800 50  0001 C CNN
+F 2 "lc_lib:stamp_2.0mm_1x10" H 9650 2800 50  0001 C CNN
 F 3 "~" H 9650 2800 50  0001 C CNN
 	1    9650 2800
@@
 F 0 "J3" H 9730 3942 50  0000 L CNN
 F 1 "Conn_01x10" H 9730 3851 50  0000 L CNN
-F 2 "Connector_PinSocket_2.00mm:PinSocket_1x10_P2.00mm_Vertical" H 9650 3950 50  0001 C CNN
+F 2 "lc_lib:stamp_2.0mm_1x10" H 9650 3950 50  0001 C CNN
 F 3 "~" H 9650 3950 50  0001 C CNN
 	1    9650 3950
@@
 F 0 "J4" H 9730 5142 50  0000 L CNN
 F 1 "Conn_01x10" H 9730 5051 50  0000 L CNN
-F 2 "Connector_PinSocket_2.00mm:PinSocket_1x10_P2.00mm_Vertical" H 9650 5150 50  0001 C CNN
+F 2 "lc_lib:stamp_2.0mm_1x10" H 9650 5150 50  0001 C CNN
 F 3 "~" H 9650 5150 50  0001 C CNN
 	1    9650 5150
