File: pcb_kicad/dap_with_general/dap-stm32f103.kicad_pcb (KiCad board)
At the start: 2 copper layers, 22 x 22 mm, 30 parts, among them J1 Conn_01x10, J2 Conn_01x10, J3 Conn_01x10, J4 Conn_01x10, U1 STM32F103CBTx, Y1 SMD-5032_2P_8MHz_20ppm_20pF

Commit message: [update] pcb general
Parts:
- added C10: 0603_10uF__106_10%_10V, lc_lib:0603_C, F.Cu at (177.0, 103.9)
- added C15: 0402_100nF__104_10%_16V, lc_lib:0402_C, F.Cu at (160.6, 99.9)
- added C9: 0402_18pF__180_5%_50V, lc_lib:0402_C, F.Cu at (157.6, 95.8)
- added D1: LED_RCBG, LED_THT:LED_D5.0mm-4_RGB, B.Cu at (159.9, 96.9)
- added G***: LOGO, Pictures:123, F.Cu at (156.9, 102.3)
- added R3: 0402_100KΩ__1003_1%, lc_lib:0402_R, F.Cu at (164.2, 100.7)
- added R4: 0402_10KΩ__1002_1%, lc_lib:0402_R, F.Cu at (166.8, 101.8)
- added SW1: SW_Push, Button_Switch_THT:SW_Tactile_SPST_Angled_PTS645Vx58-2LFS, F.Cu at (178.9, 86.7)
- added U2: STM32F103CBTx, Package_QFP:LQFP-48_7x7mm_P0.5mm, F.Cu at (171.2, 94.3)
- C5: value 0603_10uF__106_10%_10V -> 0402_100nF__104_10%_16V; footprint lc_lib:0603_C -> lc_lib:0402_C
- C6: value 0402_18pF__180_5%_50V -> 0603_10uF__106_10%_10V; footprint lc_lib:0402_C -> lc_lib:0603_C
- C7: value 0603_10uF__106_10%_10V -> 0402_18pF__180_5%_50V; footprint lc_lib:0603_C -> lc_lib:0402_C
- C8: value 0402_18pF__180_5%_50V -> 0402_100nF__104_10%_16V
- IF_SWD1: value Conn_01x05 -> Conn_01x04; footprint Connector_PinSocket_1.27mm:PinSocket_1x05_P1.27mm_Vertical -> Connector_PinHeader_2.54mm:PinHeader_1x04_P2.54mm_Vertical
- J1: value Conn_01x10 -> USB_C_Receptacle_USB2.0; footprint lc_lib:stamp_01x10_1.27mm -> Connector_USB:USB_C_Receptacle_Palconn_UTC16-G
- J2: value Conn_01x10 -> Conn_02x05_Top_Bottom; footprint lc_lib:stamp_01x10_1.27mm -> Connector_PinHeader_2.54mm:PinHeader_2x05_P2.54mm_Vertical
- J3: footprint lc_lib:stamp_01x10_1.27mm -> Connector_PinHeader_2.54mm:PinHeader_1x10_P2.54mm_Vertical
- J4: value Conn_01x10 -> Conn_01x02; footprint lc_lib:stamp_01x10_1.27mm -> Connector_PinHeader_2.54mm:PinHeader_1x02_P2.54mm_Vertical
- R10, R9: value 0402_4.7KΩ__4701_1% -> 0402_510Ω__5100_1%
- R11, R12: value 0402_33Ω__33R0_1% -> 0402_510Ω__5100_1%
- R5: value 0402_100Ω__1000_1% -> 0402_100KΩ__1003_1%
- R6: value 0402_100KΩ__1003_1% -> 0402_100Ω__1000_1%
- R7: value 0402_10KΩ__1002_1% -> 0402_33Ω__33R0_1%
- R8: value 0402_100KΩ__1003_1% -> 0402_33Ω__33R0_1%
- U1: value STM32F103CBTx -> W25Q128FVSIG_[C35101]; footprint Package_QFP:LQFP-48_7x7mm_P0.5mm -> lc_lib:SOIC-8_208MIL
- VR1: value SOT-89_HT7533-1 -> SOT-223_AMS1117-3.3; footprint lc_lib:SOT-89(SOT-89-3) -> lc_lib:SOT-223
- moved VR1 63.3 mm to (182.0, 103.6), turned to 270 degrees
- moved C14 62.3 mm to (182.1, 89.0), turned to 90 degrees
- moved C8 60.6 mm to (177.6, 105.6), turned to 180 degrees
- moved C6 56.6 mm to (177.1, 107.2), turned to 180 degrees
- moved J2 52.7 mm to (186.9, 91.3)
- moved R9 51.3 mm to (180.6, 89.0), turned to 90 degrees
- moved IF_SWD1 51.2 mm to (161.0, 106.8), turned to 270 degrees
- moved R6 51.1 mm to (184.4, 95.5), turned to 90 degrees
- moved C13 50.7 mm to (178.8, 91.6), turned to 270 degrees
- moved C11 49.8 mm to (160.6, 104.0), turned to 180 degrees
- moved C5 49.5 mm to (165.5, 89.8), turned to 315 degrees
- moved C4 49.0 mm to (176.5, 100.8), turned to 180 degrees
- moved C3 49.0 mm to (182.5, 91.6), turned to 90 degrees
- moved R1 48.7 mm to (181.0, 91.6)
- moved C1 48.5 mm to (173.3, 105.2), turned to 180 degrees
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Connections:
- C3 pad 1: GND -> /STAMP_nSRESET
- C3 pad 2: /IF_NRESET -> GND
- C4 pad 1: /STAMP_nSRESET -> GND
- C4 pad 2: GND -> /IF_NRESET
- C5 pad 1: +5V -> +3V3
- C6 pad 1: Net-(C6-Pad1) -> +5V
- C7 pad 1: +3V3 -> Net-(C7-Pad1)
- C8 pad 1: Net-(C8-Pad1) -> +5V
- IF_SWD1 pad 1: /IF_NRESET -> +3V3
- IF_SWD1 pad 2: GND -> /IF_SWDIO
- IF_SWD1 pad 3: /IF_SWCLK -> GND
- IF_SWD1 pad 4: /IF_SWDIO -> /IF_SWCLK
- J2 pad 1: GND -> +3V3
- J2 pad 10: GND -> /STAMP_UART_TX
- J2 pad 2: /STAMP_nSRESET -> GND
- J2 pad 3: /STAMP_TMS\SWDIO -> /PB10
- J2 pad 4: /STAMP_TCLK\SWCLK -> /STAMP_nSRESET
- J2 pad 5: /STAMP_TDI -> /STAMP_TMS\SWDIO
- J2 pad 6: /STAMP_TDO -> /STAMP_TCLK\SWCLK
- J2 pad 7: /STAMP_UART_TX -> /STAMP_TDI
- J2 pad 8: /STAMP_UART_RX -> /STAMP_TDO
- J2 pad 9: +3V3 -> /STAMP_UART_RX
- J3 pad 1: /PB10 -> /PB6
- J3 pad 10: GND -> /PB11
- J3 pad 2: /PB11 -> /PC14
- J3 pad 3: /PB12 -> /PC15
- J3 pad 4: /PB13 -> /PA8
- J3 pad 5: /PB14 -> /PB15
- J3 pad 6: /PB15 -> /PB14
- J3 pad 7: /PA8 -> /PB13
- J3 pad 8: /PA9 -> /PB12
- J3 pad 9: /PA10 -> /PA1
- J4 pad 1: +5V -> /IF_UART_RX
- J4 pad 2: /PB8 -> /IF_UART_TX
- R10 pad 1: Net-(R10-Pad1) -> Net-(D1-Pad1)
- R10 pad 2: GND -> /PB7
- R11 pad 1: Net-(C6-Pad1) -> Net-(D1-Pad4)
- R11 pad 2: /TGT_USB_D+ -> /PB9
- R12 pad 1: Net-(C8-Pad1) -> Net-(D1-Pad3)
- R12 pad 2: /TGT_USB_D- -> /PB8
- R5 pad 1: Net-(R5-Pad1) -> +3V3
- R5 pad 2: /STAMP_TMS\SWDIO -> /IF_NRESET
- R6 pad 1: GND -> Net-(R6-Pad1)
- R6 pad 2: Net-(R6-Pad2) -> /STAMP_TMS\SWDIO
- R7 pad 1: GND -> Net-(C7-Pad1)
- R7 pad 2: Net-(R7-Pad2) -> /TGT_USB_D+
- R8 pad 1: +3V3 -> Net-(C9-Pad1)
- R8 pad 2: /IF_NRESET -> /TGT_USB_D-
- R9 pad 1: +3V3 -> /PA0
- R9 pad 2: Net-(R10-Pad1) -> Net-(R9-Pad2)
- U1 pad 1: +3V3 -> /W25Q_CS
- U1 pad 2: Net-(R7-Pad2) -> /SPI_MISO
- U1 pad 3: /PC14 -> +3V3
- U1 pad 4: /PC15 -> GND
- U1 pad 5: Net-(C2-Pad2) -> /SPI_MOSI
- U1 pad 6: Net-(C1-Pad2) -> /SPI_SCK
- U1 pad 7: /IF_NRESET -> +3V3
- U1 pad 8: GND -> +3V3
- VR1 pad 2: +5V -> +3V3
- VR1 pad 3: +3V3 -> +5V
Routing:
- net +3V3: track 138.1 -> 195.2 mm, vias 12 -> 8
- net +5V: track 10.0 -> 64.6 mm
- net /IF_NRESET: track 37.3 -> 7.47 mm, vias 1 -> 0
- net Net-(C7-Pad1): track 0.00 -> 21.6 mm, vias 0 -> 2
- net /IF_UART_RX: track 0.00 -> 19.7 mm, vias 0 -> 1
- net GND: track 183.2 -> 202.8 mm, vias 29 -> 27
- net Net-(C9-Pad1): track 0.00 -> 19.1 mm, vias 0 -> 2
- net /IF_UART_TX: track 0.00 -> 18.8 mm, vias 0 -> 1
- net Net-(R6-Pad2): track 18.6 -> 0.00 mm, vias 2 -> 0
- net /STAMP_nSRESET: track 6.77 -> 24.3 mm
- net /IF_SWDIO: track 12.4 -> 29.5 mm, vias 2 -> 1
- net /IF_SWCLK: track 8.28 -> 25.4 mm, vias 0 -> 1
- net Net-(R2-Pad1): track 16.5 -> 2.51 mm, vias 2 -> 0
- net Net-(C8-Pad1): track 12.9 -> 0.00 mm, vias 2 -> 0
- net /W25Q_CS: track 0.00 -> 12.8 mm, vias 0 -> 2
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Other:
- board size 22 x 22 mm -> 45 x 25 mm
- board text added: "BalanceDAP"
- board text added: "GitHub:balanceTWK"
- board text added: "RT-Thread Inside"

Commit message: [update] pcb general
Other:
- board text added: "3.3V"
- board text added: "CLK"
- board text added: "DAPLink"
- board text added: "DIO"
- board text added: "DIO/TMS"
- board text added: "GND"
- board text added: "IO"
- board text added: "PA1"
- board text added: "PA8"
- board text added: "PB11"
- board text added: "PB12"
- board text added: "PB13"
- board text added: "PB14"
- board text added: "PB15"
- board text added: "PB6"
- board text added: "PC14"
- board text added: "PC15"
- board text added: "RES"
- board text added: "RX"
- board text added: "TDI"
- board text added: "TDO"
- board text added: "TX"
- board text added: "https://github.com/RT-Thread"
- board text added: "https://github.com/balanceTWK"
- board text removed: "BalanceDAP"
- board text removed: "GitHub:balanceTWK"

Commit message: [update] pcb_kicad/dap_with_general
Parts:
- moved G*** 0.24 mm to (156.6, 102.3)
Other:
- board text added: "Everything tends to balance."
- board text added: "GitHub.com/balanceTWK"
- board text added: "PCB: base on KiCad"
- board text added: "RTOS:RT-Thread inside"
- board text removed: "https://github.com/RT-Thread"
- board text removed: "https://github.com/balanceTWK"
Changed lines of the file:
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@@
-(kicad_pcb (version 20171130) (host pcbnew 5.1.4-e60b266~84~ubuntu18.04.1)
+(kicad_pcb (version 20171130) (host pcbnew "(5.1.4)-1")
   (general
     (thickness 1.6)
-    (drawings 47)
+    (drawings 49)
     (tracks 579)
     (zones 0)
@@
     (aux_axis_origin 0 0)
     (grid_origin 113.964 95.868)
-    (visible_elements FFFFFF7F)
+    (visible_elements 7FFFFFFF)
     (pcbplotparams
       (layerselection 0x010fc_ffffffff)
@@
     (add_net "Net-(R9-Pad2)")
   )
+  (module LED_THT:LED_D5.0mm-4_RGB (layer B.Cu)
+    (at 159.914 96.878)
+    (descr "LED, diameter 5.0mm, 2 pins, diameter 5.0mm, 3 pins, diameter 5.0mm, 4 pins, http://www.kingbright.com/attachments/file/psearch/000/00/00/L-154A4SUREQBFZGEW(Ver.9A).pdf")
+    (tags "LED diameter 5.0mm 2 pins diameter 5.0mm 3 pins diameter 5.0mm 4 pins RGB RGBLED")
+    (fp_text reference D1 (at 1.905 3.96) (layer B.SilkS) hide
+      (effects (font (size 1 1) (thickness 0.15)) (justify mirror))
+    )
+    (fp_text value LED_RCBG (at 1.905 -3.96) (layer B.Fab) hide
+      (effects (font (size 1 1) (thickness 0.15)) (justify mirror))
+    )
+    (fp_text user %R (at 1.905 3.96) (layer B.Fab) hide
+      (effects (font (size 1 1) (thickness 0.15)) (justify mirror))
+    )
+    (fp_line (start 5.15 3.25) (end -1.35 3.25) (layer B.CrtYd) (width 0.05))
+    (fp_line (start 5.15 -3.25) (end 5.15 3.25) (layer B.CrtYd) (width 0.05))
+    (fp_line (start -1.35 -3.25) (end 5.15 -3.25) (layer B.CrtYd) (width 0.05))
+    (fp_line (start -1.35 3.25) (end -1.35 -3.25) (layer B.CrtYd) (width 0.05))
+    (fp_line (start -0.595 1.469694) (end -0.595 -1.469694) (layer B.Fab) (width 0.1))
+    (fp_circle (center 1.905 0) (end 4.405 0) (layer B.Fab) (width 0.1))
+    (fp_arc (start 1.905 0) (end -0.595 1.469694) (angle -299.1) (layer B.Fab) (width 0.1))
+    (pad 4 thru_hole oval (at 3.81 0) (size 1.07 1.8) (drill 0.9) (layers *.Cu *.Mask)
+      (net 45 "Net-(D1-Pad4)"))
+    (pad 3 thru_hole oval (at 2.54 0) (size 1.07 1.8) (drill 0.9) (layers *.Cu *.Mask)
+      (net 46 "Net-(D1-Pad3)"))
+    (pad 2 thru_hole oval (at 1.27 0) (size 1.07 1.8) (drill 0.9) (layers *.Cu *.Mask)
+      (net 5 +3V3))
+    (pad 1 thru_hole rect (at 0 0) (size 1.07 1.8) (drill 0.9) (layers *.Cu *.Mask)
+      (net 47 "Net-(D1-Pad1)"))
+    (model ${KISYS3DMOD}/LED_THT.3dshapes/LED_D5.0mm-4_RGB.wrl
+      (at (xyz 0 0 0))
+      (scale (xyz 1 1 1))
+      (rotate (xyz 0 0 0))
+    )
+  )
   (module Pictures:123 (layer F.Cu)
-    (at 156.864 102.268)
+    (at 156.636 102.345)
     (fp_text reference G*** (at 0 0) (layer F.SilkS) hide
       (effects (font (size 1.524 1.524) (thickness 0.3)))
@@
     )
   )
-  (module LED_THT:LED_D5.0mm-4_RGB (layer B.Cu)
-    (at 159.914 96.878)
-    (descr "LED, diameter 5.0mm, 2 pins, diameter 5.0mm, 3 pins, diameter 5.0mm, 4 pins, http://www.kingbright.com/attachments/file/psearch/000/00/00/L-154A4SUREQBFZGEW(Ver.9A).pdf")
-    (tags "LED diameter 5.0mm 2 pins diameter 5.0mm 3 pins diameter 5.0mm 4 pins RGB RGBLED")
-    (fp_text reference D1 (at 1.905 3.96) (layer B.SilkS) hide
-      (effects (font (size 1 1) (thickness 0.15)))
-    )
-    (fp_text value LED_RCBG (at 1.905 -3.96) (layer B.Fab) hide
-      (effects (font (size 1 1) (thickness 0.15)) (justify mirror))
-    )
-    (fp_text user %R (at 1.905 3.96) (layer B.Fab) hide
-      (effects (font (size 1 1) (thickness 0.15)) (justify mirror))
-    )
-    (fp_line (start 5.15 3.25) (end -1.35 3.25) (layer B.CrtYd) (width 0.05))
-    (fp_line (start 5.15 -3.25) (end 5.15 3.25) (layer B.CrtYd) (width 0.05))
-    (fp_line (start -1.35 -3.25) (end 5.15 -3.25) (layer B.CrtYd) (width 0.05))
-    (fp_line (start -1.35 3.25) (end -1.35 -3.25) (layer B.CrtYd) (width 0.05))
-    (fp_line (start -0.655 -1.08) (end -0.655 -1.545) (layer B.SilkS) (width 0.12))
-    (fp_line (start -0.655 1.545) (end -0.655 1.08) (layer B.SilkS) (width 0.12))
-    (fp_line (start -0.595 1.469694) (end -0.595 -1.469694) (layer B.Fab) (width 0.1))
-    (fp_circle (center 1.905 0) (end 4.405 0) (layer B.Fab) (width 0.1))
-    (fp_arc (start 1.905 0) (end -0.349684 -1.08) (angle 128.8) (layer B.SilkS) (width 0.12))
-    (fp_arc (start 1.905 0) (end -0.349684 1.08) (angle -128.8) (layer B.SilkS) (width 0.12))
-    (fp_arc (start 1.905 0) (end -0.655 -1.54483) (angle 127.7) (layer B.SilkS) (width 0.12))
-    (fp_arc (start 1.905 0) (end -0.655 1.54483) (angle -127.7) (layer B.SilkS) (width 0.12))
-    (fp_arc (start 1.905 0) (end -0.595 1.469694) (angle -299.1) (layer B.Fab) (width 0.1))
-    (pad 4 thru_hole oval (at 3.81 0) (size 1.07 1.8) (drill 0.9) (layers *.Cu *.Mask)
-      (net 45 "Net-(D1-Pad4)"))
-    (pad 3 thru_hole oval (at 2.54 0) (size 1.07 1.8) (drill 0.9) (layers *.Cu *.Mask)
-      (net 46 "Net-(D1-Pad3)"))
-    (pad 2 thru_hole oval (at 1.27 0) (size 1.07 1.8) (drill 0.9) (layers *.Cu *.Mask)
-      (net 5 +3V3))
-    (pad 1 thru_hole rect (at 0 0) (size 1.07 1.8) (drill 0.9) (layers *.Cu *.Mask)
-      (net 47 "Net-(D1-Pad1)"))
-    (model ${KISYS3DMOD}/LED_THT.3dshapes/LED_D5.0mm-4_RGB.wrl
-      (at (xyz 0 0 0))
-      (scale (xyz 1 1 1))
-      (rotate (xyz 0 0 0))
-    )
-  )
   (module Connector_PinHeader_2.54mm:PinHeader_1x04_P2.54mm_Vertical (layer F.Cu)
     (at 161.034 106.758 270)
@@
     )
   )
+  (gr_text GitHub.com/balanceTWK (at 165.653 98.916) (layer B.SilkS)
+    (effects (font (size 1 1) (thickness 0.15)) (justify mirror))
+  )
+  (gr_text "RTOS:RT-Thread inside" (at 165.487096 93.963) (layer B.SilkS)
+    (effects (font (size 1.2 1.2) (thickness 0.15)) (justify mirror))
+  )
+  (gr_text "Everything tends to balance." (at 166.034 100.948) (layer B.SilkS)
+    (effects (font (size 1 1) (thickness 0.15) italic) (justify mirror))
+  )
+  (gr_text "PCB: base on KiCad" (at 166.715668 92.058) (layer B.SilkS)
+    (effects (font (size 1.2 1.2) (thickness 0.15)) (justify mirror))
+  )
   (gr_text PB11 (at 175.564 88.463238 90) (layer B.SilkS)
     (effects (font (size 1 1) (thickness 0.15)) (justify mirror))
@@
     (effects (font (size 1 1) (thickness 0.15)) (justify mirror))
   )
-  (gr_text https://github.com/RT-Thread (at 165.959238 92.468) (layer B.SilkS)
-    (effects (font (size 1 1) (thickness 0.15)) (justify mirror))
-  )
   (gr_text "RT-Thread Inside" (at 169.464 87.668) (layer F.SilkS)
     (effects (font (size 1 1) (thickness 0.15)))
   )
-  (gr_text https://github.com/balanceTWK (at 166.364 101.168) (layer B.SilkS)
-    (effects (font (size 1 1) (thickness 0.15)) (justify mirror))
-  )
-  (gr_text DAPLink (at 180.264 97.568) (layer F.SilkS)
+  (gr_text DAPLink (at 181.02 97.773) (layer F.SilkS)
     (effects (font (size 1.3 1.3) (thickness 0.2)))
   )

Commit message: [update] pcb general
Parts:
- removed C7, C9: 0402_18pF__180_5%_50V, lc_lib:0402_C
- removed G***: LOGO, Pictures:123
- removed IF_SWD1: Conn_01x04, Connector_PinHeader_2.54mm:PinHeader_1x04_P2.54mm_Vertical
- added R13: 0402_1.5KΩ__1501_1%, lc_lib:0402_R, F.Cu at (155.8, 98.9)
- added R14: 0402_22Ω__22R0_1%, lc_lib:0402_R, F.Cu at (155.8, 96.3)
- added R15: 0402_22Ω__22R0_1%, lc_lib:0402_R, F.Cu at (155.8, 97.5)
- added R16: 0402_0Ω__0R0_1%, lc_lib:0402_R, F.Cu at (158.0, 98.9)
- J3: value Conn_01x10 -> Conn_01x09; footprint Connector_PinHeader_2.54mm:PinHeader_1x10_P2.54mm_Vertical -> Connector_PinHeader_2.54mm:PinHeader_1x09_P2.54mm_Vertical
- J4: value Conn_01x02 -> Conn_01x06; footprint Connector_PinHeader_2.54mm:PinHeader_1x02_P2.54mm_Vertical -> Connector_PinHeader_2.54mm:PinHeader_1x06_P2.54mm_Vertical
- R5: value 0402_100KΩ__1003_1% -> 0402_10KΩ__1002_1%
- R7, R8: value 0402_33Ω__33R0_1% -> 0402_5.1KΩ__5101_1%
- moved C6 25.2 mm to (155.5, 94.1), turned to 90 degrees
- moved C10 24.2 mm to (156.3, 91.4)
- moved R10 23.7 mm to (181.4, 103.7), turned to 270 degrees
- moved C8 23.2 mm to (157.1, 94.6), turned to 90 degrees
- moved R12 22.6 mm to (182.8, 103.7), turned to 270 degrees
- moved VR1 22.3 mm to (162.4, 93.0), turned to 180 degrees
- moved D1 21.1 mm to (181.0, 96.2)
- moved R11 20.6 mm to (184.2, 103.7), turned to 270 degrees
- moved C11 19.3 mm to (179.9, 103.2), turned to 90 degrees
- moved C12 17.0 mm to (165.4, 90.2)
- moved U1 11.9 mm to (159.3, 102.9)
- moved J4 10.2 mm to (153.8, 107.2)
- moved C1 8.62 mm to (181.7, 107.4)
- moved R3 8.37 mm to (169.0, 107.6), turned to 90 degrees
- moved R8 8.15 mm to (152.2, 103.5)
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Connections:
- J1 pad A5: (no net) -> Net-(J1-PadA5)
- J1 pad B5: (no net) -> Net-(J1-PadB5)
- J2 pad 2: GND -> /PB10
- J2 pad 3: /PB10 -> /STAMP_TMS\SWDIO
- J2 pad 4: /STAMP_nSRESET -> /STAMP_TDI
- J2 pad 5: /STAMP_TMS\SWDIO -> /STAMP_UART_RX
- J2 pad 6: /STAMP_TCLK\SWCLK -> GND
- J2 pad 7: /STAMP_TDI -> /STAMP_nSRESET
- J2 pad 8: /STAMP_TDO -> /STAMP_TCLK\SWCLK
- J2 pad 9: /STAMP_UART_RX -> /STAMP_TDO
- J3 pad 1: /PB6 -> /PC14
- J3 pad 2: /PC14 -> /PC15
- J3 pad 3: /PC15 -> /PA8
- J3 pad 4: /PA8 -> /PB15
- J3 pad 5: /PB15 -> /PB14
- J3 pad 6: /PB14 -> /PB13
- J3 pad 7: /PB13 -> /PB12
- J3 pad 8: /PB12 -> /PA1
- J3 pad 9: /PA1 -> /PB11
- J4 pad 1: /IF_UART_RX -> +3V3
- J4 pad 2: /IF_UART_TX -> /IF_SWDIO
- R10 pad 2: /PB7 -> /PB9
- R11 pad 2: /PB9 -> /PB7
- R7 pad 1: Net-(C7-Pad1) -> Net-(J1-PadA5)
- R7 pad 2: /TGT_USB_D+ -> GND
- R8 pad 1: Net-(C9-Pad1) -> Net-(J1-PadB5)
- R8 pad 2: /TGT_USB_D- -> GND
- U2 pad 32: Net-(C7-Pad1) -> /MCU_USB_D-
- U2 pad 33: Net-(C9-Pad1) -> /MCU_USB_D+
Routing:
- net +5V: track 64.6 -> 14.5 mm
- net GND: track 202.8 -> 251.0 mm, vias 27 -> 16
- net Net-(C7-Pad1): track 21.6 -> 0.00 mm, vias 2 -> 0
- net Net-(C9-Pad1): track 19.1 -> 0.00 mm, vias 2 -> 0
- net /IF_SWCLK: track 25.4 -> 11.5 mm
- net /IF_SWDIO: track 29.5 -> 16.0 mm
- net /PB8: track 4.89 -> 17.1 mm, vias 0 -> 2
- net /MCU_USB_D-: track 0.00 -> 11.9 mm
- net /PB7: track 7.59 -> 19.4 mm
- net /MCU_USB_D+: track 0.00 -> 11.5 mm
- net +3V3: track 195.2 -> 184.3 mm, vias 8 -> 12
- net /PB9: track 4.69 -> 15.0 mm, vias 0 -> 2
- net Net-(J1-PadA5): track 0.00 -> 7.31 mm, vias 0 -> 2
- net /IF_UART_RX: track 19.7 -> 12.5 mm
- net Net-(J1-PadB5): track 0.00 -> 6.77 mm
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- removed copper zone on B.Cu, net GND
- removed copper zone on F.Cu, net GND

Commit message: [update] pcb general
Routing:
- added copper zone on B.Cu, net GND
- added copper zone on F.Cu, net GND
Other:
- board text removed: "PB6"

Commit message: [update] pcb
Parts:
- added G***: LOGO, Pictures:github, F.Cu at (182.5, 99.9)

Commit message: [update] PCB
Parts:
- moved G*** 3.50 mm to (179.0, 99.8)
Other:
- board text added: "BalanceDAP"
- board text added: "PCB: KiCad"
- board text added: "RTOS:RT-Thread"
- board text removed: "DAPLink"
- board text removed: "PCB: base on KiCad"
- board text removed: "RT-Thread Inside"
- board text removed: "RTOS:RT-Thread inside"
Changed lines of the file:
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@@
   (general
     (thickness 1.6)
-    (drawings 50)
+    (drawings 49)
     (tracks 602)
     (zones 0)
@@
   )
   (module Pictures:github (layer F.Cu)
-    (at 182.464 99.868)
+    (at 178.964 99.768)
     (fp_text reference G*** (at 0 0) (layer F.SilkS) hide
       (effects (font (size 1.524 1.524) (thickness 0.3)))
@@
   (gr_line (start 179.764 90.668) (end 179.764 103.068) (layer B.SilkS) (width 0.12))
   (gr_line (start 168.964 103.068) (end 168.964 90.668) (layer B.SilkS) (width 0.12))
-  (gr_text "RT-Thread Inside" (at 165.214 88.118) (layer F.SilkS)
-    (effects (font (size 1 1) (thickness 0.15)))
-  )
-  (gr_text DAPLink (at 171.214 90.618) (layer F.SilkS)
+  (gr_text BalanceDAP (at 165.664 88.068) (layer F.SilkS)
     (effects (font (size 1.3 1.3) (thickness 0.2)))
   )
@@
     (effects (font (size 1 1) (thickness 0.15)) (justify mirror))
   )
-  (gr_text "RTOS:RT-Thread inside" (at 157.737096 96.96) (layer B.SilkS)
+  (gr_text RTOS:RT-Thread (at 160.537096 97.26) (layer B.SilkS)
     (effects (font (size 1.2 1.2) (thickness 0.15)) (justify mirror))
   )
-  (gr_text "Everything tends to balance." (at 157.214 98.618) (layer B.SilkS)
+  (gr_text "Everything tends to balance." (at 156.94662 98.918) (layer B.SilkS)
     (effects (font (size 1 1) (thickness 0.15) italic) (justify mirror))
   )
-  (gr_text "PCB: base on KiCad" (at 158.965668 95.308) (layer B.SilkS)
+  (gr_text "PCB: KiCad" (at 162.737096 95.608) (layer B.SilkS)
     (effects (font (size 1.2 1.2) (thickness 0.15)) (justify mirror))
   )
@@
     (effects (font (size 1 1) (thickness 0.15)) (justify mirror))
   )
-  (gr_text CLK (at 153.964 104.139428 90) (layer B.SilkS)
+  (gr_text CLK (at 161.464 104.139428 90) (layer B.SilkS)
     (effects (font (size 1 1) (thickness 0.15)) (justify mirror))
   )
-  (gr_text GND (at 156.484 104.020381 90) (layer B.SilkS)
+  (gr_text GND (at 158.964 104.020381 90) (layer B.SilkS)
     (effects (font (size 1 1) (thickness 0.15)) (justify mirror))
   )
-  (gr_text DIO (at 159.004 104.282285 90) (layer B.SilkS)
+  (gr_text DIO (at 156.214 104.282285 90) (layer B.SilkS)
     (effects (font (size 1 1) (thickness 0.15)) (justify mirror))
   )
-  (gr_text 3.3V (at 161.524 103.925143 90) (layer B.SilkS)
+  (gr_text 3.3V (at 153.714 103.925143 90) (layer B.SilkS)
     (effects (font (size 1 1) (thickness 0.15)) (justify mirror))
   )
